Commit message: Update

File: robotics_demo/scripts/ur5v2/ur5_robot.urdf (robot description, URDF)
Before this commit: robot ur5, 10 links, 9 joints
Joints:
- joint shoulder_lift_joint: origin xyz=0.0 0.13585 0.0 rpy=0.0 1.570796325 0.0 -> xyz=0.0 0.13585 0.0 rpy=0.0 0.0 0.0
- joint wrist_1_joint: origin xyz=0.0 0.0 0.39225 rpy=0.0 1.570796325 0.0 -> xyz=0.0 0.0 0.39225 rpy=0.0 0.0 0.0
